File: kicad/power.sch (KiCad schematic (older format))
At the start: 6 parts, among them J1 Conn_02x05_Odd_Even, U8 L7805

Commit message: Work on schematics and pcbs.
Connections:
- net +12V: now also J1.10 (Pin_10), J1.9 (Pin_9); no longer J1.1 (Pin_1), J1.2 (Pin_2)
Changed lines of the file:
@@
 $Descr A4 11693 8268
 encoding utf-8
-Sheet 5 3
+Sheet 2 2
 Title ""
 Date ""
@@
 L power:+12V #PWR0104
 U 1 1 5CFAD59E
-P 3750 5300
-F 0 "#PWR0104" H 3750 5150 50  0001 C CNN
-F 1 "+12V" V 3765 5428 50  0000 L CNN
-F 2 "" H 3750 5300 50  0001 C CNN
-F 3 "" H 3750 5300 50  0001 C CNN
-	1    3750 5300
+P 3800 5700
+F 0 "#PWR0104" H 3800 5550 50  0001 C CNN
+F 1 "+12V" V 3815 5828 50  0000 L CNN
+F 2 "" H 3800 5700 50  0001 C CNN
+F 3 "" H 3800 5700 50  0001 C CNN
+	1    3800 5700
 	0    -1   -1   0
 $EndComp
@@
 L power:+12V #PWR0105
 U 1 1 5CFAD5B5
-P 4350 5300
-F 0 "#PWR0105" H 4350 5150 50  0001 C CNN
-F 1 "+12V" V 4365 5428 50  0000 L CNN
-F 2 "" H 4350 5300 50  0001 C CNN
-F 3 "" H 4350 5300 50  0001 C CNN
-	1    4350 5300
+P 4300 5700
+F 0 "#PWR0105" H 4300 5550 50  0001 C CNN
+F 1 "+12V" V 4315 5828 50  0000 L CNN
+F 2 "" H 4300 5700 50  0001 C CNN
+F 3 "" H 4300 5700 50  0001 C CNN
+	1    4300 5700
 	0    1    1    0
 $EndComp
@@
 Wire Wire Line
 	3800 5600 3800 5500
-Wire Wire Line
-	3800 5300 3750 5300
-Wire Wire Line
-	4350 5300 4300 5300
-NoConn ~ 4300 5700
-NoConn ~ 3800 5700
 $Comp
 L power:+5V #PWR?
@@
 	6000 3450 5950 3450
 Connection ~ 5950 3450
+NoConn ~ 4300 5300
+NoConn ~ 3800 5300
 $EndSCHEMATC

Commit message: Work on pcbs a bit.
Parts:
- R77, R78: footprint Resistor_SMD:R_1206_3216Metric_Pad1.42x1.75mm_HandSolder -> Resistor_SMD:R_0805_2012Metric_Pad1.15x1.40mm_HandSolder
Changed lines of the file:
@@
 F 0 "R77" H 7820 3496 50  0000 L CNN
 F 1 "2K2" H 7820 3405 50  0000 L CNN
-F 2 "Resistor_SMD:R_1206_3216Metric_Pad1.42x1.75mm_HandSolder" V 7680 3450 50  0001 C CNN
+F 2 "Resistor_SMD:R_0805_2012Metric_Pad1.15x1.40mm_HandSolder" V 7680 3450 50  0001 C CNN
 F 3 "~" H 7750 3450 50  0001 C CNN
 	1    7750 3450
@@
 F 0 "R78" H 7820 3896 50  0000 L CNN
 F 1 "3K3" H 7820 3805 50  0000 L CNN
-F 2 "Resistor_SMD:R_1206_3216Metric_Pad1.42x1.75mm_HandSolder" V 7680 3850 50  0001 C CNN
+F 2 "Resistor_SMD:R_0805_2012Metric_Pad1.15x1.40mm_HandSolder" V 7680 3850 50  0001 C CNN
 F 3 "~" H 7750 3850 50  0001 C CNN
 	1    7750 3850

Commit message: More work on pcbs and frontpanel.
Parts:
- removed R77: 2K2, Resistor_SMD:R_0805_2012Metric_Pad1.15x1.40mm_HandSolder, symbol Device:R
- removed R78: 3K3, Resistor_SMD:R_0805_2012Metric_Pad1.15x1.40mm_HandSolder, symbol Device:R
- removed U8: L7805, Package_TO_SOT_THT:TO-220-3_Horizontal_TabDown, symbol Regulator_Linear:L7805
- added C1, C2: C, Capacitor_SMD:CP_Elec_5x3.9, symbol Device:C
- added D1, D2: D, Diode_SMD:D_0805_2012Metric_Pad1.15x1.40mm_HandSolder, symbol Device:D
- added U1: LD1117S50TR_SOT223, Package_TO_SOT_SMD:SOT-223-3_TabPin2, symbol Regulator_Linear:LD1117S50TR_SOT223
- added U2: LD1117S33TR_SOT223, Package_TO_SOT_SMD:SOT-223-3_TabPin2, symbol Regulator_Linear:LD1117S33TR_SOT223
- C17, C18: footprint Capacitor_SMD:C_1206_3216Metric_Pad1.42x1.75mm_HandSolder -> Capacitor_SMD:CP_Elec_5x3.9
Connections:
- net +12V: now also D2.2 (A); no longer C17.1
- net +3V3: now also C2.1, U2.2 (VO)
- net GND: now also C1.2, C2.2, U1.1 (GND), U2.1 (GND)
- net +5V: no longer names the net of C18.1
- net +5V: now also D1.2 (A), U1.2 (VO)
- new net: C17.1, D2.1 (K), U1.3 (VI)
- new net CA7_VCC: C1.1, D1.1 (K), U2.3 (VI)
Other:
- moved on the sheet: C17, C18
Changed lines of the file:
@@
 	2750 3400 2650 3400
-$Comp
-L Regulator_Linear:L7805 U8
-U 1 1 5CF7E36B
-P 5600 3450
-F 0 "U8" H 5600 3692 50  0000 C CNN
-F 1 "L7805" H 5600 3601 50  0000 C CNN
-F 2 "Package_TO_SOT_THT:TO-220-3_Horizontal_TabDown" H 5625 3300 50  0001 L CIN
-F 3 "http://www.st.com/content/ccc/resource/technical/document/datasheet/41/4f/b3/b0/12/d4/47/88/CD00000444.pdf/files/CD00000444.pdf/jcr:content/translations/en.CD00000444.pdf" H 5600 3400 50  0001 C CNN
-	1    5600 3450
-	1    0    0    -1
-$EndComp
 $Comp
 L power:+12V #PWR052
 U 1 1 5CF7E486
-P 5150 3450
-F 0 "#PWR052" H 5150 3300 50  0001 C CNN
-F 1 "+12V" V 5165 3578 50  0000 L CNN
-F 2 "" H 5150 3450 50  0001 C CNN
-F 3 "" H 5150 3450 50  0001 C CNN
-	1    5150 3450
+P 4350 3450
+F 0 "#PWR052" H 4350 3300 50  0001 C CNN
+F 1 "+12V" V 4365 3578 50  0000 L CNN
+F 2 "" H 4350 3450 50  0001 C CNN
+F 3 "" H 4350 3450 50  0001 C CNN
+	1    4350 3450
 	0    -1   -1   0
 $EndComp
@@
 L power:GND #PWR?
 U 1 1 5CF7E4D8
-P 5600 4000
+P 5100 4000
 AR Path="/5CF7E4D8" Ref="#PWR?"  Part="1"
 AR Path="/5CF3B46A/5CF7E4D8" Ref="#PWR053"  Part="1"
-F 0 "#PWR053" H 5600 3750 50  0001 C CNN
-F 1 "GND" V 5605 3872 50  0000 R CNN
-F 2 "" H 5600 4000 50  0001 C CNN
-F 3 "" H 5600 4000 50  0001 C CNN
-	1    5600 4000
+F 0 "#PWR053" H 5100 3750 50  0001 C CNN
+F 1 "GND" V 5105 3872 50  0000 R CNN
+F 2 "" H 5100 4000 50  0001 C CNN
+F 3 "" H 5100 4000 50  0001 C CNN
+	1    5100 4000
 	1    0    0    -1
 $EndComp
@@
 L Device:C C17
 U 1 1 5CF7E50F
-P 5250 3800
-F 0 "C17" H 5365 3846 50  0000 L CNN
-F 1 "C" H 5365 3755 50  0000 L CNN
-F 2 "Capacitor_SMD:C_1206_3216Metric_Pad1.42x1.75mm_HandSolder" H 5288 3650 50  0001 C CNN
-F 3 "~" H 5250 3800 50  0001 C CNN
-	1    5250 3800
+P 4750 3800
+F 0 "C17" H 4865 3846 50  0000 L CNN
+F 1 "C" H 4865 3755 50  0000 L CNN
+F 2 "Capacitor_SMD:CP_Elec_5x3.9" H 4788 3650 50  0001 C CNN
+F 3 "~" H 4750 3800 50  0001 C CNN
+	1    4750 3800
 	1    0    0    -1
 $EndComp
@@
 L Device:C C18
 U 1 1 5CF7E55B
-P 5950 3800
-F 0 "C18" H 6065 3846 50  0000 L CNN
-F 1 "C" H 6065 3755 50  0000 L CNN
-F 2 "Capacitor_SMD:C_1206_3216Metric_Pad1.42x1.75mm_HandSolder" H 5988 3650 50  0001 C CNN
-F 3 "~" H 5950 3800 50  0001 C CNN
-	1    5950 3800
-	1    0    0    -1
-$EndComp
-Wire Wire Line
-	5250 3950 5600 3950
-Wire Wire Line
-	5600 4000 5600 3950
-Connection ~ 5600 3950
-Wire Wire Line
-	5600 3950 5950 3950
-Wire Wire Line
-	5600 3750 5600 3950
-Wire Wire Line
-	5900 3450 5950 3450
-Wire Wire Line
-	5950 3650 5950 3450
-Wire Wire Line
-	5250 3650 5250 3450
-Wire Wire Line
-	5250 3450 5300 3450
-Wire Wire Line
-	5150 3450 5250 3450
-Connection ~ 5250 3450
-$Comp
-L power:GND #PWR?
-U 1 1 5CF7EB2C
-P 7750 4050
-AR Path="/5CF7EB2C" Ref="#PWR?"  Part="1"
-AR Path="/5CF3B46A/5CF7EB2C" Ref="#PWR056"  Part="1"
-F 0 "#PWR056" H 7750 3800 50  0001 C CNN
-F 1 "GND" V 7755 3922 50  0000 R CNN
-F 2 "" H 7750 4050 50  0001 C CNN
-F 3 "" H 7750 4050 50  0001 C CNN
-	1    7750 4050
-	1    0    0    -1
-$EndComp
-$Comp
-L Device:R R77
-U 1 1 5CF7EB6E
-P 7750 3450
-F 0 "R77" H 7820 3496 50  0000 L CNN
-F 1 "2K2" H 7820 3405 50  0000 L CNN
-F 2 "Resistor_SMD:R_0805_2012Metric_Pad1.15x1.40mm_HandSolder" V 7680 3450 50  0001 C CNN
-F 3 "~" H 7750 3450 50  0001 C CNN
-	1    7750 3450
-	1    0    0    -1
-$EndComp
-$Comp
-L Device:R R78
-U 1 1 5CF7EBA6
-P 7750 3850
-F 0 "R78" H 7820 3896 50  0000 L CNN
-F 1 "3K3" H 7820 3805 50  0000 L CNN
-F 2 "Resistor_SMD:R_0805_2012Metric_Pad1.15x1.40mm_HandSolder" V 7680 3850 50  0001 C CNN
-F 3 "~" H 7750 3850 50  0001 C CNN
-	1    7750 3850
-	1    0    0    -1
-$EndComp
-$Comp
-L power:+3.3V #PWR?
-U 1 1 5CF7EC1D
-P 8000 3650
-AR Path="/5CF7EC1D" Ref="#PWR?"  Part="1"
-AR Path="/5CF3B46A/5CF7EC1D" Ref="#PWR057"  Part="1"
-F 0 "#PWR057" H 8000 3500 50  0001 C CNN
-F 1 "+3.3V" H 8015 3823 50  0000 C CNN
-F 2 "" H 8000 3650 50  0001 C CNN
-F 3 "" H 8000 3650 50  0001 C CNN
-	1    8000 3650
-	0    1    1    0
-$EndComp
-Wire Wire Line
-	8000 3650 7750 3650
-Wire Wire Line
-	7750 3650 7750 3700
-Wire Wire Line
-	7750 3600 7750 3650
-Connection ~ 7750 3650
-Wire Wire Line
-	7750 4050 7750 4000
-Wire Wire Line
-	7750 3250 7750 3300
+P 5450 3800
+F 0 "C18" H 5565 3846 50  0000 L CNN
+F 1 "C" H 5565 3755 50  0000 L CNN
+F 2 "Capacitor_SMD:CP_Elec_5x3.9" H 5488 3650 50  0001 C CNN
+F 3 "~" H 5450 3800 50  0001 C CNN
+	1    5450 3800
+	1    0    0    -1
+$EndComp
+Wire Wire Line
+	4750 3950 5100 3950
+Wire Wire Line
+	5100 4000 5100 3950
+Connection ~ 5100 3950
+Wire Wire Line
+	5100 3950 5450 3950
+Wire Wire Line
+	5100 3750 5100 3950
+Wire Wire Line
+	5400 3450 5450 3450
+Wire Wire Line
+	5450 3650 5450 3450
+Wire Wire Line
+	4750 3650 4750 3450
+Wire Wire Line
+	4750 3450 4800 3450
+Wire Wire Line
+	4650 3450 4750 3450
+Connection ~ 4750 3450
 Wire Wire Line
 	2850 3800 2650 3800
@@
 Wire Wire Line
 	3800 5600 3800 5500
-$Comp
-L power:+5V #PWR?
-U 1 1 5CFF1B04
-P 7750 3250
-AR Path="/5CFF1B04" Ref="#PWR?"  Part="1"
-AR Path="/5CF3B46A/5CFF1B04" Ref="#PWR0106"  Part="1"
-F 0 "#PWR0106" H 7750 3100 50  0001 C CNN
-F 1 "+5V" V 7765 3378 50  0000 L CNN
-F 2 "" H 7750 3250 50  0001 C CNN
-F 3 "" H 7750 3250 50  0001 C CNN
-	1    7750 3250
-	1    0    0    -1
-$EndComp
-$Comp
-L power:+5V #PWR?
-U 1 1 5CFF1E84
-P 6000 3450
-AR Path="/5CFF1E84" Ref="#PWR?"  Part="1"
-AR Path="/5CF3B46A/5CFF1E84" Ref="#PWR0107"  Part="1"
-F 0 "#PWR0107" H 6000 3300 50  0001 C CNN
-F 1 "+5V" V 6015 3578 50  0000 L CNN
-F 2 "" H 6000 3450 50  0001 C CNN
-F 3 "" H 6000 3450 50  0001 C CNN
-	1    6000 3450
-	0    1    1    0
-$EndComp
-Wire Wire Line
-	6000 3450 5950 3450
-Connection ~ 5950 3450
+Connection ~ 5450 3450
 NoConn ~ 4300 5300
 NoConn ~ 3800 5300
+$Comp
+L Regulator_Linear:LD1117S33TR_SOT223 U2
+U 1 1 5E1180B9
+P 6800 3450
+F 0 "U2" H 6800 3692 50  0000 C CNN
+F 1 "LD1117S33TR_SOT223" H 6800 3601 50  0000 C CNN
+F 2 "Package_TO_SOT_SMD:SOT-223-3_TabPin2" H 6800 3650 50  0001 C CNN
+F 3 "http://www.st.com/st-web-ui/static/active/en/resource/technical/document/datasheet/CD00000544.pdf" H 6900 3200 50  0001 C CNN
+	1    6800 3450
+	1    0    0    -1
+$EndComp
+$Comp
+L Regulator_Linear:LD1117S50TR_SOT223 U1
+U 1 1 5E1181EC
+P 5100 3450
+F 0 "U1" H 5100 3692 50  0000 C CNN
+F 1 "LD1117S50TR_SOT223" H 5100 3601 50  0000 C CNN
+F 2 "Package_TO_SOT_SMD:SOT-223-3_TabPin2" H 5100 3650 50  0001 C CNN
+F 3 "http://www.st.com/st-web-ui/static/active/en/resource/technical/document/datasheet/CD00000544.pdf" H 5200 3200 50  0001 C CNN
+	1    5100 3450
+	1    0    0    -1
+$EndComp
+Wire Wire Line
+	5450 3450 5700 3450
+Wire Wire Line
+	6200 3200 6200 3450
+Wire Wire Line
+	6200 3450 6400 3450
+$Comp
+L power:+3.3V #PWR?
+U 1 1 5E119369
+P 7250 3450
+AR Path="/5E119369" Ref="#PWR?"  Part="1"
+AR Path="/5CF3B46A/5E119369" Ref="#PWR01"  Part="1"
+F 0 "#PWR01" H 7250 3300 50  0001 C CNN
+F 1 "+3.3V" H 7265 3623 50  0000 C CNN
+F 2 "" H 7250 3450 50  0001 C CNN
+F 3 "" H 7250 3450 50  0001 C CNN
+	1    7250 3450
+	0    1    1    0
+$EndComp
+$Comp
+L Device:C C1
+U 1 1 5E119454
+P 6400 3800
+F 0 "C1" H 6515 3846 50  0000 L CNN
+F 1 "C" H 6515 3755 50  0000 L CNN
+F 2 "Capacitor_SMD:CP_Elec_5x3.9" H 6438 3650 50  0001 C CNN
+F 3 "~" H 6400 3800 50  0001 C CNN
+	1    6400 3800
+	1    0    0    -1
+$EndComp
+$Comp
+L Device:C C2
+U 1 1 5E11949E
+P 7150 3800
+F 0 "C2" H 7265 3846 50  0000 L CNN
+F 1 "C" H 7265 3755 50  0000 L CNN
+F 2 "Capacitor_SMD:CP_Elec_5x3.9" H 7188 3650 50  0001 C CNN
+F 3 "~" H 7150 3800 50  0001 C CNN
+	1    7150 3800
+	1    0    0    -1
+$EndComp
+Wire Wire Line
+	7250 3450 7150 3450
+Wire Wire Line
+	7150 3650 7150 3450
+Connection ~ 7150 3450
+Wire Wire Line
+	7150 3450 7100 3450
+Wire Wire Line
+	6400 3650 6400 3450
+Connection ~ 6400 3450
+Wire Wire Line
+	6400 3450 6500 3450
+$Comp
+L power:GND #PWR?
+U 1 1 5E11A2E0
+P 6800 4000
+AR Path="/5E11A2E0" Ref="#PWR?"  Part="1"
+AR Path="/5CF3B46A/5E11A2E0" Ref="#PWR02"  Part="1"
+F 0 "#PWR02" H 6800 3750 50  0001 C CNN
+F 1 "GND" V 6805 3872 50  0000 R CNN
+F 2 "" H 6800 4000 50  0001 C CNN
+F 3 "" H 6800 4000 50  0001 C CNN
+	1    6800 4000
+	1    0    0    -1
+$EndComp
+Wire Wire Line
+	6800 3750 6800 3950
+Connection ~ 6800 3950
+Wire Wire Line
+	6800 3950 7150 3950
+Wire Wire Line
+	6800 3950 6800 4000
+Wire Wire Line
+	6400 3950 6800 3950
+$Comp
+L Device:D D2
+U 1 1 5E11B11F
+P 4500 3450
+F 0 "D2" H 4500 3234 50  0000 C CNN
+F 1 "D" H 4500 3325 50  0000 C CNN
+F 2 "Diode_SMD:D_0805_2012Metric_Pad1.15x1.40mm_HandSolder" H 4500 3450 50  0001 C CNN
+F 3 "~" H 4500 3450 50  0001 C CNN
+	1    4500 3450
+	-1   0    0    1
+$EndComp
+Text GLabel 6200 3200 1    50   Input ~ 0
+CA7_VCC
+$Comp
+L Device:D D1
+U 1 1 5E120B83
+P 5850 3450
+F 0 "D1" H 5850 3234 50  0000 C CNN
+F 1 "D" H 5850 3325 50  0000 C CNN
+F 2 "Diode_SMD:D_0805_2012Metric_Pad1.15x1.40mm_HandSolder" H 5850 3450 50  0001 C CNN
+F 3 "~" H 5850 3450 50  0001 C CNN
+	1    5850 3450
+	-1   0    0    1
+$EndComp
+Wire Wire Line
+	6000 3450 6200 3450
+Connection ~ 6200 3450
 $EndSCHEMATC

Commit message: Work on base pcb/schematics + frontpanel.
Parts:
- C1, C17: footprint Capacitor_SMD:CP_Elec_5x3.9 -> Capacitor_SMD:CP_Elec_6.3x7.7
- C18, C2: footprint Capacitor_SMD:CP_Elec_5x3.9 -> Capacitor_SMD:CP_Elec_5x5.4
- D1, D2: footprint Diode_SMD:D_0805_2012Metric_Pad1.15x1.40mm_HandSolder -> Diode_SMD:D_SMA
Changed lines of the file:
@@
 F 0 "C17" H 4865 3846 50  0000 L CNN
 F 1 "C" H 4865 3755 50  0000 L CNN
-F 2 "Capacitor_SMD:CP_Elec_5x3.9" H 4788 3650 50  0001 C CNN
+F 2 "Capacitor_SMD:CP_Elec_6.3x7.7" H 4788 3650 50  0001 C CNN
 F 3 "~" H 4750 3800 50  0001 C CNN
 	1    4750 3800
@@
 F 0 "C18" H 5565 3846 50  0000 L CNN
 F 1 "C" H 5565 3755 50  0000 L CNN
-F 2 "Capacitor_SMD:CP_Elec_5x3.9" H 5488 3650 50  0001 C CNN
+F 2 "Capacitor_SMD:CP_Elec_5x5.4" H 5488 3650 50  0001 C CNN
 F 3 "~" H 5450 3800 50  0001 C CNN
 	1    5450 3800
@@
 F 0 "C1" H 6515 3846 50  0000 L CNN
 F 1 "C" H 6515 3755 50  0000 L CNN
-F 2 "Capacitor_SMD:CP_Elec_5x3.9" H 6438 3650 50  0001 C CNN
+F 2 "Capacitor_SMD:CP_Elec_6.3x7.7" H 6438 3650 50  0001 C CNN
 F 3 "~" H 6400 3800 50  0001 C CNN
 	1    6400 3800
@@
 F 0 "C2" H 7265 3846 50  0000 L CNN
 F 1 "C" H 7265 3755 50  0000 L CNN
-F 2 "Capacitor_SMD:CP_Elec_5x3.9" H 7188 3650 50  0001 C CNN
+F 2 "Capacitor_SMD:CP_Elec_5x5.4" H 7188 3650 50  0001 C CNN
 F 3 "~" H 7150 3800 50  0001 C CNN
 	1    7150 3800
@@
 F 0 "D2" H 4500 3234 50  0000 C CNN
 F 1 "D" H 4500 3325 50  0000 C CNN
-F 2 "Diode_SMD:D_0805_2012Metric_Pad1.15x1.40mm_HandSolder" H 4500 3450 50  0001 C CNN
+F 2 "Diode_SMD:D_SMA" H 4500 3450 50  0001 C CNN
 F 3 "~" H 4500 3450 50  0001 C CNN
 	1    4500 3450
@@
 F 0 "D1" H 5850 3234 50  0000 C CNN
 F 1 "D" H 5850 3325 50  0000 C CNN
-F 2 "Diode_SMD:D_0805_2012Metric_Pad1.15x1.40mm_HandSolder" H 5850 3450 50  0001 C CNN
+F 2 "Diode_SMD:D_SMA" H 5850 3450 50  0001 C CNN
 F 3 "~" H 5850 3450 50  0001 C CNN
 	1    5850 3450
