File: kicad/midirouter.kicad_pcb (KiCad board)
At the start: 2 copper layers, 152.9 x 47.2 mm, 33 parts, among them J1 Conn_02x05_Odd_Even, J2 Conn_01x08, J3 Conn_01x08, J4 Conn_01x08, J5 Conn_01x08, J6 Conn_01x08, J7 Conn_01x08, J8 Conn_01x08, J9 Conn_01x08, Q1 PN2222A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

Commit message: Work on schematics and pcbs.
Parts:
- U5, U6: footprint Package_SO:SOP-16_7.5x10.4mm_P1.27mm -> Package_SO:SOP-16_4.4x10.4mm_P1.27mm
- moved U6 1.91 mm to (67.3, 62.9)
- moved U5 1.02 mm to (170.2, 67.3)
Connections:
- J1 pad 1: +12V -> Net-(J1-Pad1)
- J1 pad 10: Net-(J1-Pad10) -> +12V
- J1 pad 2: +12V -> Net-(J1-Pad2)
- J1 pad 9: Net-(J1-Pad9) -> +12V
Routing:
- net Net-(U5-Pad11): track 0.00 -> 125.5 mm, vias 0 -> 3
- net +5V: track 123.8 -> 0.00 mm
- net Net-(U5-Pad12): track 0.00 -> 121.3 mm, vias 0 -> 3
- net Net-(U5-Pad9): track 0.00 -> 113.0 mm, vias 0 -> 2
- net LED1: track 91.8 -> 148.5 mm, vias 1 -> 2
- net LED2: track 92.5 -> 144.7 mm, vias 1 -> 2
- net LED3: track 92.0 -> 140.7 mm, vias 1 -> 2
- net LED4: track 94.1 -> 139.2 mm
- net LED5: track 0.00 -> 23.3 mm
- net LED6: track 0.00 -> 21.6 mm
- net LED7: track 0.00 -> 19.1 mm
- net GND: track 0.00 -> 17.8 mm
- net LED8: track 0.00 -> 17.0 mm
- net Net-(R17-Pad2): track 0.00 -> 13.4 mm
- net Net-(R24-Pad2): track 0.00 -> 7.14 mm
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- added copper zone on B.Cu, net GND
- added copper zone on F.Cu, net GND

Commit message: Work on pcbs a bit.
Parts:
- Q1, Q2, Q3, Q4: footprint Package_TO_SOT_THT:TO-92_Inline -> Tomarus:MMBT2222A-SOT23
- R17, R18, R19, R20, R21, R22, R23, R24, R25, R26, R27, R28, R77, R78: footprint Resistor_SMD:R_1206_3216Metric_Pad1.42x1.75mm_HandSolder -> Resistor_SMD:R_0805_2012Metric_Pad1.15x1.40mm_HandSolder
- U5, U6: value 74LS594 -> 74LS595
- moved R17 23.4 mm to (162.0, 52.0), turned to 270 degrees
- moved R18 21.3 mm to (164.0, 52.0), turned to 270 degrees
- moved R19 19.6 mm to (166.0, 52.0), turned to 270 degrees
- moved R20 18.1 mm to (168.0, 52.0), turned to 270 degrees
- moved R24 17.2 mm to (176.0, 52.0), turned to 270 degrees
- moved R21 17.1 mm to (170.0, 52.0), turned to 270 degrees
- moved R23 16.6 mm to (174.0, 52.0), turned to 270 degrees
- moved R22 16.6 mm to (172.0, 52.0), turned to 270 degrees
- moved U5 8.72 mm to (168.9, 58.7), turned to 270 degrees
- moved R77 1.84 mm to (41.8, 83.5), turned to 270 degrees
- moved R78 1.74 mm to (47.0, 83.5), turned to 90 degrees
- moved Q4 1.42 mm to (59.2, 73.2), turned to 90 degrees
- moved Q3 1.33 mm to (64.8, 73.2), turned to 90 degrees
- moved Q2 1.24 mm to (70.2, 73.2), turned to 90 degrees
- moved Q1 1.15 mm to (75.8, 73.2), turned to 90 degrees
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Connections:
- U5 pad 13: +3V3 -> GND
- U6 pad 13: +3V3 -> GND
Routing:
- net GND: track 17.8 -> 39.0 mm, vias 0 -> 8
- net Net-(U5-Pad11): track 125.5 -> 111.5 mm, vias 3 -> 2
- net Net-(U5-Pad12): track 121.3 -> 108.5 mm, vias 3 -> 0
- net LED5: track 23.3 -> 11.8 mm
- net +3V3: track 246.2 -> 235.2 mm, vias 4 -> 6
- net LED6: track 21.6 -> 11.3 mm
- net LED7: track 19.1 -> 10.9 mm
- net LED8: track 17.0 -> 10.2 mm
- net +5V: track 0.00 -> 6.18 mm
- net LED1: track 148.5 -> 143.0 mm
- net LED2: track 144.7 -> 140.4 mm
- net +12V: track 24.4 -> 27.8 mm
- net Net-(R17-Pad2): track 13.4 -> 10.4 mm
- net Net-(R18-Pad2): track 5.70 -> 2.71 mm
- net Net-(U5-Pad9): track 113.0 -> 110.1 mm, vias 2 -> 0
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Other:
- board text added: "R17-R24"

Commit message: More work on pcbs and frontpanel.
Parts:
- removed R77: 2K2, Resistor_SMD:R_0805_2012Metric_Pad1.15x1.40mm_HandSolder
- removed R78: 3K3, Resistor_SMD:R_0805_2012Metric_Pad1.15x1.40mm_HandSolder
- removed U8: L7805, Package_TO_SOT_THT:TO-220-3_Horizontal_TabDown
- added C1: C, Capacitor_SMD:CP_Elec_5x3.9, B.Cu at (41.5, 65.0)
- added C2: C, Capacitor_SMD:CP_Elec_5x3.9, B.Cu at (41.5, 77.0)
- added D1: D, Diode_SMD:D_0805_2012Metric_Pad1.15x1.40mm_HandSolder, B.Cu at (48.0, 68.0)
- added D2: D, Diode_SMD:D_0805_2012Metric_Pad1.15x1.40mm_HandSolder, B.Cu at (47.5, 56.0)
- added U1: LD1117S50TR_SOT223, Package_TO_SOT_SMD:SOT-223-3_TabPin2, B.Cu at (51.0, 62.0)
- added U2: LD1117S33TR_SOT223, Package_TO_SOT_SMD:SOT-223-3_TabPin2, B.Cu at (51.0, 74.0)
- C17, C18: footprint Capacitor_SMD:C_1206_3216Metric_Pad1.42x1.75mm_HandSolder -> Capacitor_SMD:CP_Elec_5x3.9
- moved R25 103.4 mm to (162.0, 79.0)
- moved Q4 102.1 mm to (161.0, 82.2)
- moved R26 101.9 mm to (166.0, 79.0)
- moved Q3 101.6 mm to (166.0, 82.2)
- moved Q2 101.2 mm to (171.0, 82.2)
- moved U6 100.9 mm to (167.8, 71.9)
- moved Q1 100.7 mm to (176.0, 82.2)
- moved R27 100.4 mm to (170.0, 79.0)
- moved R28 98.9 mm to (174.0, 79.0)
- moved C17 21.8 mm to (41.5, 59.0)
- moved U7 19.0 mm to (78.0, 67.0)
- moved C18 8.91 mm to (41.5, 71.0), turned to 180 degrees
- moved R17 2.24 mm to (161.0, 54.0)
- moved R18 2.24 mm to (163.0, 54.0)
- moved R19 2.24 mm to (165.0, 54.0)
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Connections:
- C17 pad 1: +12V -> Net-(C17-Pad1)
- C18 pad 1: +5V -> Net-(C18-Pad1)
- U7 pad 24: +5V -> CA7_VCC
Routing:
- net CA7_VCC: track 0.00 -> 108.0 mm
- net Net-(U5-Pad9): track 110.1 -> 5.99 mm
- net LED8: track 10.2 -> 112.2 mm, vias 0 -> 2
- net LED5: track 11.8 -> 106.4 mm, vias 0 -> 3
- net LED7: track 10.9 -> 105.2 mm, vias 0 -> 3
- net LED6: track 11.3 -> 104.9 mm, vias 0 -> 3
- net LEDK2: track 68.9 -> 139.4 mm, vias 1 -> 3
- net LEDK1: track 67.1 -> 135.5 mm, vias 0 -> 3
- net Net-(U5-Pad14): track 0.00 -> 55.0 mm
- net Net-(U5-Pad12): track 108.5 -> 55.8 mm, vias 0 -> 2
- net Net-(U5-Pad11): track 111.5 -> 61.9 mm
- net LEDK3: track 105.6 -> 59.1 mm, vias 1 -> 2
- net LEDK4: track 104.5 -> 61.6 mm, vias 0 -> 2
- net GND: track 39.0 -> 79.4 mm, vias 8 -> 7
- net MIDI_IN_12: track 18.2 -> 39.1 mm
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- removed copper zone on B.Cu, net GND
Other:
- board size 152.9 x 47.2 mm -> 153.5 x 49 mm

Commit message: Work on base pcb/schematics + frontpanel.
Parts:
- added C3: 100n, Capacitor_SMD:C_0805_2012Metric, B.Cu at (161.2, 63.0)
- added C4: 100n, Capacitor_SMD:C_0805_2012Metric, B.Cu at (174.5, 69.5)
- C1, C17: footprint Capacitor_SMD:CP_Elec_5x3.9 -> Capacitor_SMD:CP_Elec_6.3x7.7
- C18, C2: footprint Capacitor_SMD:CP_Elec_5x3.9 -> Capacitor_SMD:CP_Elec_5x5.4
- D1, D2: footprint Diode_SMD:D_0805_2012Metric_Pad1.15x1.40mm_HandSolder -> Diode_SMD:D_SMA
- moved C18 7.02 mm to (42.0, 64.0)
- moved C1 6.03 mm to (41.8, 71.0)
- moved D2 3.82 mm to (50.8, 58.0), turned to 180 degrees
- moved D1 3.26 mm to (50.8, 69.8)
- moved U1 2.15 mm to (52.2, 63.8)
- moved U2 2.15 mm to (52.2, 75.8)
- moved C17 2.02 mm to (41.8, 57.0)
- moved C2 1.13 mm to (42.0, 78.0)
Routing:
- net GND: track 79.4 -> 95.4 mm, vias 7 -> 10
- net CA7_VCC: track 108.0 -> 96.3 mm
- net +3V3: track 253.5 -> 260.3 mm
- net Net-(C17-Pad1): track 7.29 -> 12.9 mm
- net +12V: track 21.4 -> 24.7 mm
- net MIDI_OUT_1: track 43.0 -> 45.9 mm
- net Net-(R17-Pad2): track 13.0 -> 15.5 mm
- net Net-(C18-Pad1): track 18.5 -> 20.8 mm
- net MIDI_OUT_2: track 44.2 -> 45.9 mm
- net MIDI_OUT_4: track 46.9 -> 46.0 mm
- net MIDI_OUT_3: track 45.2 -> 45.9 mm
Other:
- board text added: "JLCJLCJLCJLC"
- board text added: "MIDI Merger Bus Board v1.0 github.com/tomarus/midirouter"

Commit message: Updates to frontpanels, schematics and pcbs.
Other:
- board text added: "."
