File: kicad/midiboard/midirouter.kicad_pcb (KiCad board)
At the start: 2 copper layers, 39 x 85 mm, 59 parts, among them J1 MIDI_IN_1, J10 Conn_01x08, J2 MIDI_IN_2, J3 MIDI_IN_3, J4 MIDI_IN_4, J5 Conn_01x08, J6 MIDI_OUT_1, J7 MIDI_OUT_2, J8 MIDI_OUT_3, J9 MIDI_OUT_4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

Commit message: Silkscreen and text updates.
Other:
- board text added: "JLCJLCJLCJLC"
- board text added: "MIDI ROUTER 4xDIN-5 IO BOARD v1.0 github.com/tomarus/midirouter"
Changed lines of the file:
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@@
   (general
     (thickness 1.6)
-    (drawings 14)
+    (drawings 16)
     (tracks 370)
     (zones 0)
@@
     )
   )
+  (gr_text "MIDI ROUTER \n4xDIN-5 IO BOARD v1.0\ngithub.com/tomarus/midirouter" (at 95 148.25) (layer B.SilkS)
+    (effects (font (size 1 1) (thickness 0.15)) (justify mirror))
+  )
+  (gr_text JLCJLCJLCJLC (at 95 150) (layer F.SilkS)
+    (effects (font (size 1 1) (thickness 0.15)))
+  )
   (gr_text . (at 93.25 108.75) (layer B.SilkS)

Commit message: Some minor silkscreen updates.
Other:
- board text added: "MIDI ROUTER 4xDIN5 IO BOARD v1.0 github.com/tomarus/midirouter"
- board text removed: "MIDI ROUTER 4xDIN-5 IO BOARD v1.0 github.com/tomarus/midirouter"
Changed lines of the file:
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@@
     (visible_elements FFFFFF7F)
     (pcbplotparams
-      (layerselection 0x010fc_ffffffff)
+      (layerselection 0x010f0_ffffffff)
       (usegerberextensions false)
       (usegerberattributes false)
@@
       (outputformat 1)
       (mirror false)
-      (drillshape 1)
+      (drillshape 0)
       (scaleselection 1)
-      (outputdirectory ""))
+      (outputdirectory "Gerbers"))
   )
   (net 0 "")
@@
     )
   )
-  (gr_text "MIDI ROUTER \n4xDIN-5 IO BOARD v1.0\ngithub.com/tomarus/midirouter" (at 95 148.25) (layer B.SilkS)
+  (gr_text "MIDI ROUTER \n4xDIN5 IO BOARD v1.0\ngithub.com/tomarus/midirouter" (at 95 148.25) (layer B.SilkS)
     (effects (font (size 1 1) (thickness 0.15)) (justify mirror))
   )
